Commit message: Add tempo imitation for debugging and many other changes

File: models/humanMeshed/robots/humanMeshed.urdf (robot description, URDF)
Before this commit: robot humanMeshed, 61 links, 60 joints
Links:
- added link left_toe_pitch
- added link left_toe_roll
- added link left_toe_yaw
- added link right_toe_pitch
- added link right_toe_roll
- added link right_toe_yaw
- link chest_yaw: geometry visual mesh filename=package://online_tempo/models/humanMeshed/meshes/chest.dae scale=0.06 0.06 0.06
- link head_yaw: geometry visual mesh filename=package://online_tempo/models/humanMeshed/meshes/head.dae scale=0.06 0.06 0.06
- link hip_yaw: geometry visual mesh filename=package://online_tempo/models/humanMeshed/meshes/pelvis.dae scale=0.06 0.06 0.06
- link left_clavicle_yaw: geometry visual mesh filename=package://online_tempo/models/humanMeshed/meshes/leftClavic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 scale=0.06 0.06 0.06
- link left_elbow_yaw: geometry visual mesh filename=package://online_tempo/models/humanMeshed/meshes/leftForear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 scale=0.06 0.06 0.06
- link left_foot_yaw: geometry visual mesh filename=package://online_tempo/models/humanMeshed/meshes/leftFoot.d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 scale=0.06 0.06 0.06
- link left_hand_yaw: geometry visual mesh filename=package://online_tempo/models/humanMeshed/meshes/leftHand.d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 scale=0.06 0.06 0.06
- link left_knee_yaw: geometry visual mesh filename=package://online_tempo/models/humanMeshed/meshes/leftShin.d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 scale=0.06 0.06 0.06
- link left_shoulder_yaw: geometry visual mesh filename=package://online_tempo/models/humanMeshed/meshes/leftBicep.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 scale=0.06 0.06 0.06
- link left_thigh_yaw: geometry visual mesh filename=package://online_tempo/models/humanMeshed/meshes/leftThigh.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 scale=0.06 0.06 0.06
- link lower_spine_yaw: geometry visual mesh filename=package://online_tempo/models/humanMeshed/meshes/abdomen.dae scale=0.06 0.06 0.06
- link middle_spine_yaw: geometry 
- link neck_yaw: geometry visual mesh filename=package://online_tempo/models/humanMeshed/meshes/neck.dae scale=0.06 0.06 0.06
- link right_clavicle_yaw: geometry visual mesh filename=package://online_tempo/models/humanMeshed/meshes/rightClavi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 scale=0.06 0.06 0.06
- link right_elbow_yaw: geometry visual mesh filename=package://online_tempo/models/humanMeshed/meshes/rightForea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 scale=0.06 0.06 0.06
- link right_foot_yaw: geometry visual mesh filename=package://online_tempo/models/humanMeshed/meshes/rightFoot.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 scale=0.06 0.06 0.06
- link right_hand_yaw: geometry visual mesh filename=package://online_tempo/models/humanMeshed/meshes/rightHand.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 scale=0.06 0.06 0.06
- link right_knee_yaw: geometry visual mesh filename=package://online_tempo/models/humanMeshed/meshes/rightShin.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 scale=0.06 0.06 0.06
- link right_shoulder_yaw: geometry visual mesh filename=package://online_tempo/models/humanMeshed/meshes/rightBicep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 scale=0.06 0.06 0.06
- link right_thigh_yaw: geometry visual mesh filename=package://online_tempo/models/humanMeshed/meshes/rightThigh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 scale=0.06 0.06 0.06
Joints:
- added joint left_toe_pitch: type continuous, parent left_toe_roll, child left_toe_pitch, origin xyz=0 0 0, axis 0 1.0 0
- added joint left_toe_roll: type continuous, parent left_foot_yaw, child left_toe_roll, origin xyz=0.11 0.0025 -0.07, axis 1.0 0 0
- added joint left_toe_yaw: type continuous, parent left_toe_pitch, child left_toe_yaw, origin xyz=0 0 0, axis 0 0 1.0
- added joint right_toe_pitch: type continuous, parent right_toe_roll, child right_toe_pitch, origin xyz=0 0 0, axis 0 1.0 0
- added joint right_toe_roll: type continuous, parent right_foot_yaw, child right_toe_roll, origin xyz=0.11 -0.0025 -0.07, axis 1.0 0 0
- added joint right_toe_yaw: type continuous, parent right_toe_pitch, child right_toe_yaw, origin xyz=0 0 0, axis 0 0 1.0
- joint hip_roll: origin xyz=0 0 0.90 -> xyz=0.05 0 0.90
- joint left_clavicle_roll: origin xyz=0 0.0125 0.22 -> xyz=-0.04 0.0125 0.22
- joint left_elbow_roll: origin xyz=0 0.27 0 -> xyz=0 0.23 -0.095
- joint left_foot_roll: origin xyz=0 0 -0.43 -> xyz=-0.0225 -0.0125 -0.425
- joint left_hand_roll: origin xyz=0 0.24 0 -> xyz=0.046 0.211 -0.04
- joint left_knee_roll: origin xyz=0 0 -0.43 -> xyz=-0.05 -0.02 -0.3375
- joint left_shoulder_roll: origin xyz=0 0.135 0 -> xyz=0 0.16 0.0225
- joint left_thigh_roll: origin xyz=0 0.175 0 -> xyz=0 0.0875 -0.0875
- joint neck_roll: origin xyz=0 0 0.22 -> xyz=0 0 0.25
- joint right_clavicle_roll: origin xyz=0 -0.0125 0.22 -> xyz=-0.04 -0.0125 0.22
- joint right_elbow_roll: origin xyz=0 -0.27 0 -> xyz=0 -0.23 -0.095
- joint right_foot_roll: origin xyz=0 0 -0.43 -> xyz=-0.0225 0.0125 -0.425
- joint right_hand_roll: origin xyz=0 -0.24 0 -> xyz=0.046 -0.211 -0.04
- joint right_knee_roll: origin xyz=0 0 -0.43 -> xyz=-0.05 0.02 -0.3375
- joint right_shoulder_roll: origin xyz=0 -0.135 0 -> xyz=0 -0.16 0.0225
- joint right_thigh_roll: origin xyz=0 -0.175 0 -> xyz=0 -0.0875 -0.0875
