Commit message: Rename online_tempo to rostango in every file

File: models/humanMeshed/robots/abomination.urdf (robot description, URDF)
Before this commit: robot humanMeshed, 89 links, 88 joints
Links:
- link chest_yaw: geometry visual mesh filename=package://rostango/models/humanMeshed/meshes/chest.dae scale=0.06 0.06 0.06
- link head_yaw: geometry visual mesh filename=package://rostango/models/humanMeshed/meshes/head.dae scale=0.06 0.06 0.06
- link hip_yaw: geometry visual mesh filename=package://rostango/models/humanMeshed/meshes/pelvis.dae scale=0.06 0.06 0.06
- link left_clavicle_yaw: geometry visual mesh filename=package://rostango/models/humanMeshed/meshes/leftClavicle.d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 scale=0.06 0.06 0.06
- link left_elbow_yaw: geometry visual mesh filename=package://rostango/models/humanMeshed/meshes/leftForearm.dae scale=0.06 0.06 0.06
- link left_foot_yaw: geometry visual mesh filename=package://rostango/models/humanMeshed/meshes/leftFoot.dae scale=0.06 0.06 0.06
- link left_hand_yaw: geometry visual mesh filename=package://rostango/models/humanMeshed/meshes/leftHand.dae scale=0.06 0.06 0.06
- link left_knee_yaw: geometry visual mesh filename=package://rostango/models/humanMeshed/meshes/leftShin.dae scale=0.06 0.06 0.06
- link left_shoulder_yaw: geometry visual mesh filename=package://rostango/models/humanMeshed/meshes/leftBicep.dae scale=0.06 0.06 0.06
- link left_thigh_yaw: geometry visual mesh filename=package://rostango/models/humanMeshed/meshes/leftThigh.dae scale=0.06 0.06 0.06
- link lower_spine_yaw: geometry visual mesh filename=package://rostango/models/humanMeshed/meshes/abdomen.dae scale=0.06 0.06 0.06
- link neck_yaw: geometry visual mesh filename=package://rostango/models/humanMeshed/meshes/neck.dae scale=0.06 0.06 0.06
- link right_clavicle_yaw: geometry visual mesh filename=package://rostango/models/humanMeshed/meshes/rightClavicle.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 scale=0.06 0.06 0.06
- link right_elbow_yaw: geometry visual mesh filename=package://rostango/models/humanMeshed/meshes/rightForearm.d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 scale=0.06 0.06 0.06
- link right_foot_yaw: geometry visual mesh filename=package://rostango/models/humanMeshed/meshes/rightFoot.dae scale=0.06 0.06 0.06
- link right_hand_yaw: geometry visual mesh filename=package://rostango/models/humanMeshed/meshes/rightHand.dae scale=0.06 0.06 0.06
- link right_knee_yaw: geometry visual mesh filename=package://rostango/models/humanMeshed/meshes/rightShin.dae scale=0.06 0.06 0.06
- link right_shoulder_yaw: geometry visual mesh filename=package://rostango/models/humanMeshed/meshes/rightBicep.dae scale=0.06 0.06 0.06
- link right_thigh_yaw: geometry visual mesh filename=package://rostango/models/humanMeshed/meshes/rightThigh.dae scale=0.06 0.06 0.06

File: models/humanMeshed/robots/abominationv2.urdf (robot description, URDF)
Before this commit: robot humanMeshed, 89 links, 88 joints
Links:
- link chest_yaw: geometry visual mesh filename=package://rostango/models/humanMeshed/meshes/chest.dae scale=0.06 0.06 0.06
- link head_yaw: geometry visual mesh filename=package://rostango/models/humanMeshed/meshes/head.dae scale=0.06 0.06 0.06
- link hip_yaw: geometry visual mesh filename=package://rostango/models/humanMeshed/meshes/pelvis.dae scale=0.06 0.06 0.06
- link left_clavicle_yaw: geometry visual mesh filename=package://rostango/models/humanMeshed/meshes/leftClavicle.d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 scale=0.06 0.06 0.06
- link left_elbow_yaw: geometry visual mesh filename=package://rostango/models/humanMeshed/meshes/leftForearm.dae scale=0.06 0.06 0.06
- link left_foot_yaw: geometry visual mesh filename=package://rostango/models/humanMeshed/meshes/leftFoot.dae scale=0.06 0.06 0.06
- link left_hand_yaw: geometry visual mesh filename=package://rostango/models/humanMeshed/meshes/leftHand.dae scale=0.06 0.06 0.06
- link left_knee_yaw: geometry visual mesh filename=package://rostango/models/humanMeshed/meshes/leftShin.dae scale=0.06 0.06 0.06
- link left_shoulder_yaw: geometry visual mesh filename=package://rostango/models/humanMeshed/meshes/leftBicep.dae scale=0.06 0.06 0.06
- link left_thigh_yaw: geometry visual mesh filename=package://rostango/models/humanMeshed/meshes/leftThigh.dae scale=0.06 0.06 0.06
- link lower_spine_yaw: geometry visual mesh filename=package://rostango/models/humanMeshed/meshes/abdomen.dae scale=0.06 0.06 0.06
- link neck_yaw: geometry visual mesh filename=package://rostango/models/humanMeshed/meshes/neck.dae scale=0.06 0.06 0.06
- link right_clavicle_yaw: geometry visual mesh filename=package://rostango/models/humanMeshed/meshes/rightClavicle.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 scale=0.06 0.06 0.06
- link right_elbow_yaw: geometry visual mesh filename=package://rostango/models/humanMeshed/meshes/rightForearm.d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 scale=0.06 0.06 0.06
- link right_foot_yaw: geometry visual mesh filename=package://rostango/models/humanMeshed/meshes/rightFoot.dae scale=0.06 0.06 0.06
- link right_hand_yaw: geometry visual mesh filename=package://rostango/models/humanMeshed/meshes/rightHand.dae scale=0.06 0.06 0.06
- link right_knee_yaw: geometry visual mesh filename=package://rostango/models/humanMeshed/meshes/rightShin.dae scale=0.06 0.06 0.06
- link right_shoulder_yaw: geometry visual mesh filename=package://rostango/models/humanMeshed/meshes/rightBicep.dae scale=0.06 0.06 0.06
- link right_thigh_yaw: geometry visual mesh filename=package://rostango/models/humanMeshed/meshes/rightThigh.dae scale=0.06 0.06 0.06

File: models/humanMeshed/robots/humanDefaultOdom.urdf (robot description, URDF)
Before this commit: robot humanMeshed, 68 links, 67 joints
Links:
- link chest_yaw: geometry visual mesh filename=package://rostango/models/humanMeshed/meshes/chest.dae scale=0.06 0.06 0.06
- link head_yaw: geometry visual mesh filename=package://rostango/models/humanMeshed/meshes/head.dae scale=0.06 0.06 0.06
- link hip_yaw: geometry visual mesh filename=package://rostango/models/humanMeshed/meshes/pelvis.dae scale=0.06 0.06 0.06
- link left_clavicle_yaw: geometry visual mesh filename=package://rostango/models/humanMeshed/meshes/leftClavicle.d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 scale=0.06 0.06 0.06
- link left_elbow_yaw: geometry visual mesh filename=package://rostango/models/humanMeshed/meshes/leftForearm.dae scale=0.06 0.06 0.06
- link left_foot_yaw: geometry visual mesh filename=package://rostango/models/humanMeshed/meshes/leftFoot.dae scale=0.06 0.06 0.06
- link left_hand_yaw: geometry visual mesh filename=package://rostango/models/humanMeshed/meshes/leftHand.dae scale=0.06 0.06 0.06
- link left_knee_yaw: geometry visual mesh filename=package://rostango/models/humanMeshed/meshes/leftShin.dae scale=0.06 0.06 0.06
- link left_shoulder_yaw: geometry visual mesh filename=package://rostango/models/humanMeshed/meshes/leftBicep.dae scale=0.06 0.06 0.06
- link left_thigh_yaw: geometry visual mesh filename=package://rostango/models/humanMeshed/meshes/leftThigh.dae scale=0.06 0.06 0.06
- link lower_spine_yaw: geometry visual mesh filename=package://rostango/models/humanMeshed/meshes/abdomen.dae scale=0.06 0.06 0.06
- link neck_yaw: geometry visual mesh filename=package://rostango/models/humanMeshed/meshes/neck.dae scale=0.06 0.06 0.06
- link right_clavicle_yaw: geometry visual mesh filename=package://rostango/models/humanMeshed/meshes/rightClavicle.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 scale=0.06 0.06 0.06
- link right_elbow_yaw: geometry visual mesh filename=package://rostango/models/humanMeshed/meshes/rightForearm.d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 scale=0.06 0.06 0.06
- link right_foot_yaw: geometry visual mesh filename=package://rostango/models/humanMeshed/meshes/rightFoot.dae scale=0.06 0.06 0.06
- link right_hand_yaw: geometry visual mesh filename=package://rostango/models/humanMeshed/meshes/rightHand.dae scale=0.06 0.06 0.06
- link right_knee_yaw: geometry visual mesh filename=package://rostango/models/humanMeshed/meshes/rightShin.dae scale=0.06 0.06 0.06
- link right_shoulder_yaw: geometry visual mesh filename=package://rostango/models/humanMeshed/meshes/rightBicep.dae scale=0.06 0.06 0.06
- link right_thigh_yaw: geometry visual mesh filename=package://rostango/models/humanMeshed/meshes/rightThigh.dae scale=0.06 0.06 0.06

File: models/humanMeshed/robots/humanMeshed.urdf (robot description, URDF)
Before this commit: robot humanMeshed, 67 links, 66 joints
Links:
- link chest_yaw: geometry visual mesh filename=package://rostango/models/humanMeshed/meshes/chest.dae scale=0.06 0.06 0.06
- link head_yaw: geometry visual mesh filename=package://rostango/models/humanMeshed/meshes/head.dae scale=0.06 0.06 0.06
- link hip_yaw: geometry visual mesh filename=package://rostango/models/humanMeshed/meshes/pelvis.dae scale=0.06 0.06 0.06
- link left_clavicle_yaw: geometry visual mesh filename=package://rostango/models/humanMeshed/meshes/leftClavicle.d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 scale=0.06 0.06 0.06
- link left_elbow_yaw: geometry visual mesh filename=package://rostango/models/humanMeshed/meshes/leftForearm.dae scale=0.06 0.06 0.06
- link left_foot_yaw: geometry visual mesh filename=package://rostango/models/humanMeshed/meshes/leftFoot.dae scale=0.06 0.06 0.06
- link left_hand_yaw: geometry visual mesh filename=package://rostango/models/humanMeshed/meshes/leftHand.dae scale=0.06 0.06 0.06
- link left_knee_yaw: geometry visual mesh filename=package://rostango/models/humanMeshed/meshes/leftShin.dae scale=0.06 0.06 0.06
- link left_shoulder_yaw: geometry visual mesh filename=package://rostango/models/humanMeshed/meshes/leftBicep.dae scale=0.06 0.06 0.06
- link left_thigh_yaw: geometry visual mesh filename=package://rostango/models/humanMeshed/meshes/leftThigh.dae scale=0.06 0.06 0.06
- link lower_spine_yaw: geometry visual mesh filename=package://rostango/models/humanMeshed/meshes/abdomen.dae scale=0.06 0.06 0.06
- link neck_yaw: geometry visual mesh filename=package://rostango/models/humanMeshed/meshes/neck.dae scale=0.06 0.06 0.06
- link right_clavicle_yaw: geometry visual mesh filename=package://rostango/models/humanMeshed/meshes/rightClavicle.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 scale=0.06 0.06 0.06
- link right_elbow_yaw: geometry visual mesh filename=package://rostango/models/humanMeshed/meshes/rightForearm.d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 scale=0.06 0.06 0.06
- link right_foot_yaw: geometry visual mesh filename=package://rostango/models/humanMeshed/meshes/rightFoot.dae scale=0.06 0.06 0.06
- link right_hand_yaw: geometry visual mesh filename=package://rostango/models/humanMeshed/meshes/rightHand.dae scale=0.06 0.06 0.06
- link right_knee_yaw: geometry visual mesh filename=package://rostango/models/humanMeshed/meshes/rightShin.dae scale=0.06 0.06 0.06
- link right_shoulder_yaw: geometry visual mesh filename=package://rostango/models/humanMeshed/meshes/rightBicep.dae scale=0.06 0.06 0.06
- link right_thigh_yaw: geometry visual mesh filename=package://rostango/models/humanMeshed/meshes/rightThigh.dae scale=0.06 0.06 0.06

File: models/humanMeshed/robots/humanMeshedAligned.urdf (robot description, URDF)
Before this commit: robot humanMeshed, 67 links, 66 joints
Links:
- link chest_yaw: geometry visual mesh filename=package://rostango/models/humanMeshed/meshes/chest.dae scale=0.06 0.06 0.06
- link head_yaw: geometry visual mesh filename=package://rostango/models/humanMeshed/meshes/head.dae scale=0.06 0.06 0.06
- link hip_yaw: geometry visual mesh filename=package://rostango/models/humanMeshed/meshes/pelvis.dae scale=0.06 0.06 0.06
- link left_clavicle_yaw: geometry visual mesh filename=package://rostango/models/humanMeshed/meshes/leftClavicle.d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 scale=0.06 0.06 0.06
- link left_elbow_yaw: geometry visual mesh filename=package://rostango/models/humanMeshed/meshes/leftForearm.dae scale=0.06 0.06 0.06
- link left_foot_yaw: geometry visual mesh filename=package://rostango/models/humanMeshed/meshes/leftFoot.dae scale=0.06 0.06 0.06
- link left_hand_yaw: geometry visual mesh filename=package://rostango/models/humanMeshed/meshes/leftHand.dae scale=0.06 0.06 0.06
- link left_knee_yaw: geometry visual mesh filename=package://rostango/models/humanMeshed/meshes/leftShin.dae scale=0.06 0.06 0.06
- link left_shoulder_yaw: geometry visual mesh filename=package://rostango/models/humanMeshed/meshes/leftBicep.dae scale=0.06 0.06 0.06
- link left_thigh_yaw: geometry visual mesh filename=package://rostango/models/humanMeshed/meshes/leftThigh.dae scale=0.06 0.06 0.06
- link lower_spine_yaw: geometry visual mesh filename=package://rostango/models/humanMeshed/meshes/abdomen.dae scale=0.06 0.06 0.06
- link neck_yaw: geometry visual mesh filename=package://rostango/models/humanMeshed/meshes/neck.dae scale=0.06 0.06 0.06
- link right_clavicle_yaw: geometry visual mesh filename=package://rostango/models/humanMeshed/meshes/rightClavicle.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 scale=0.06 0.06 0.06
- link right_elbow_yaw: geometry visual mesh filename=package://rostango/models/humanMeshed/meshes/rightForearm.d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 scale=0.06 0.06 0.06
- link right_foot_yaw: geometry visual mesh filename=package://rostango/models/humanMeshed/meshes/rightFoot.dae scale=0.06 0.06 0.06
- link right_hand_yaw: geometry visual mesh filename=package://rostango/models/humanMeshed/meshes/rightHand.dae scale=0.06 0.06 0.06
- link right_knee_yaw: geometry visual mesh filename=package://rostango/models/humanMeshed/meshes/rightShin.dae scale=0.06 0.06 0.06
- link right_shoulder_yaw: geometry visual mesh filename=package://rostango/models/humanMeshed/meshes/rightBicep.dae scale=0.06 0.06 0.06
- link right_thigh_yaw: geometry visual mesh filename=package://rostango/models/humanMeshed/meshes/rightThigh.dae scale=0.06 0.06 0.06

File: models/humanMeshed/robots/humanMeshedModified.urdf (robot description, URDF)
Before this commit: robot humanMeshed, 89 links, 88 joints
Links:
- link chest_yaw: geometry visual mesh filename=package://rostango/models/humanMeshed/meshes/chest.dae scale=0.06 0.06 0.06
- link head_yaw: geometry visual mesh filename=package://rostango/models/humanMeshed/meshes/head.dae scale=0.06 0.06 0.06
- link hip_yaw: geometry visual mesh filename=package://rostango/models/humanMeshed/meshes/pelvis.dae scale=0.06 0.06 0.06
- link left_clavicle_yaw: geometry visual mesh filename=package://rostango/models/humanMeshed/meshes/leftClavicle.d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 scale=0.06 0.06 0.06
- link left_elbow_yaw: geometry visual mesh filename=package://rostango/models/humanMeshed/meshes/leftForearm.dae scale=0.06 0.06 0.06
- link left_foot_yaw: geometry visual mesh filename=package://rostango/models/humanMeshed/meshes/leftFoot.dae scale=0.06 0.06 0.06
- link left_hand_yaw: geometry visual mesh filename=package://rostango/models/humanMeshed/meshes/leftHand.dae scale=0.06 0.06 0.06
- link left_knee_yaw: geometry visual mesh filename=package://rostango/models/humanMeshed/meshes/leftShin.dae scale=0.06 0.06 0.06
- link left_shoulder_yaw: geometry visual mesh filename=package://rostango/models/humanMeshed/meshes/leftBicep.dae scale=0.06 0.06 0.06
- link left_thigh_yaw: geometry visual mesh filename=package://rostango/models/humanMeshed/meshes/leftThigh.dae scale=0.06 0.06 0.06
- link lower_spine_yaw: geometry visual mesh filename=package://rostango/models/humanMeshed/meshes/abdomen.dae scale=0.06 0.06 0.06
- link neck_yaw: geometry visual mesh filename=package://rostango/models/humanMeshed/meshes/neck.dae scale=0.06 0.06 0.06
- link right_clavicle_yaw: geometry visual mesh filename=package://rostango/models/humanMeshed/meshes/rightClavicle.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 scale=0.06 0.06 0.06
- link right_elbow_yaw: geometry visual mesh filename=package://rostango/models/humanMeshed/meshes/rightForearm.d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 scale=0.06 0.06 0.06
- link right_foot_yaw: geometry visual mesh filename=package://rostango/models/humanMeshed/meshes/rightFoot.dae scale=0.06 0.06 0.06
- link right_hand_yaw: geometry visual mesh filename=package://rostango/models/humanMeshed/meshes/rightHand.dae scale=0.06 0.06 0.06
- link right_knee_yaw: geometry visual mesh filename=package://rostango/models/humanMeshed/meshes/rightShin.dae scale=0.06 0.06 0.06
- link right_shoulder_yaw: geometry visual mesh filename=package://rostango/models/humanMeshed/meshes/rightBicep.dae scale=0.06 0.06 0.06
- link right_thigh_yaw: geometry visual mesh filename=package://rostango/models/humanMeshed/meshes/rightThigh.dae scale=0.06 0.06 0.06

File: models/humanMeshed/robots/humanMeshedv2.urdf (robot description, URDF)
Before this commit: robot humanMeshed, 67 links, 66 joints
Links:
- link chest_yaw: geometry visual mesh filename=package://rostango/models/humanMeshed/meshes/chest.dae scale=0.06 0.06 0.06
- link head_yaw: geometry visual mesh filename=package://rostango/models/humanMeshed/meshes/head.dae scale=0.06 0.06 0.06
- link hip_yaw: geometry visual mesh filename=package://rostango/models/humanMeshed/meshes/pelvis.dae scale=0.06 0.06 0.06
- link left_clavicle_yaw: geometry visual mesh filename=package://rostango/models/humanMeshed/meshes/leftClavicle.d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 scale=0.06 0.06 0.06
- link left_elbow_yaw: geometry visual mesh filename=package://rostango/models/humanMeshed/meshes/leftForearm.dae scale=0.06 0.06 0.06
- link left_foot_yaw: geometry visual mesh filename=package://rostango/models/humanMeshed/meshes/leftFoot.dae scale=0.06 0.06 0.06
- link left_hand_yaw: geometry visual mesh filename=package://rostango/models/humanMeshed/meshes/leftHand.dae scale=0.06 0.06 0.06
- link left_knee_yaw: geometry visual mesh filename=package://rostango/models/humanMeshed/meshes/leftShin.dae scale=0.06 0.06 0.06
- link left_shoulder_yaw: geometry visual mesh filename=package://rostango/models/humanMeshed/meshes/leftBicep.dae scale=0.06 0.06 0.06
- link left_thigh_yaw: geometry visual mesh filename=package://rostango/models/humanMeshed/meshes/leftThigh.dae scale=0.06 0.06 0.06
- link lower_spine_yaw: geometry visual mesh filename=package://rostango/models/humanMeshed/meshes/abdomen.dae scale=0.06 0.06 0.06
- link neck_yaw: geometry visual mesh filename=package://rostango/models/humanMeshed/meshes/neck.dae scale=0.06 0.06 0.06
- link right_clavicle_yaw: geometry visual mesh filename=package://rostango/models/humanMeshed/meshes/rightClavicle.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 scale=0.06 0.06 0.06
- link right_elbow_yaw: geometry visual mesh filename=package://rostango/models/humanMeshed/meshes/rightForearm.d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 scale=0.06 0.06 0.06
- link right_foot_yaw: geometry visual mesh filename=package://rostango/models/humanMeshed/meshes/rightFoot.dae scale=0.06 0.06 0.06
- link right_hand_yaw: geometry visual mesh filename=package://rostango/models/humanMeshed/meshes/rightHand.dae scale=0.06 0.06 0.06
- link right_knee_yaw: geometry visual mesh filename=package://rostango/models/humanMeshed/meshes/rightShin.dae scale=0.06 0.06 0.06
- link right_shoulder_yaw: geometry visual mesh filename=package://rostango/models/humanMeshed/meshes/rightBicep.dae scale=0.06 0.06 0.06
- link right_thigh_yaw: geometry visual mesh filename=package://rostango/models/humanMeshed/meshes/rightThigh.dae scale=0.06 0.06 0.06

File: models/humanMeshed/robots/humanModifiedOdom.urdf (robot description, URDF)
Before this commit: robot humanMeshed, 90 links, 89 joints
Links:
- link chest_yaw: geometry visual mesh filename=package://rostango/models/humanMeshed/meshes/chest.dae scale=0.06 0.06 0.06
- link head_yaw: geometry visual mesh filename=package://rostango/models/humanMeshed/meshes/head.dae scale=0.06 0.06 0.06
- link hip_yaw: geometry visual mesh filename=package://rostango/models/humanMeshed/meshes/pelvis.dae scale=0.06 0.06 0.06
- link left_clavicle_yaw: geometry visual mesh filename=package://rostango/models/humanMeshed/meshes/leftClavicle.d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 scale=0.06 0.06 0.06
- link left_elbow_yaw: geometry visual mesh filename=package://rostango/models/humanMeshed/meshes/leftForearm.dae scale=0.062 0.06 0.06
- link left_foot_yaw: geometry visual mesh filename=package://rostango/models/humanMeshed/meshes/leftFoot.dae scale=0.06 0.06 0.06
- link left_hand_yaw: geometry visual mesh filename=package://rostango/models/humanMeshed/meshes/leftHand.dae scale=0.06 0.06 0.06
- link left_knee_yaw: geometry visual mesh filename=package://rostango/models/humanMeshed/meshes/leftShin.dae scale=0.06 0.06 0.06
- link left_shoulder_yaw: geometry visual mesh filename=package://rostango/models/humanMeshed/meshes/leftBicep.dae scale=0.07 0.06 0.06
- link left_thigh_yaw: geometry visual mesh filename=package://rostango/models/humanMeshed/meshes/leftThigh.dae scale=0.06 0.06 0.06
- link lower_spine_yaw: geometry visual mesh filename=package://rostango/models/humanMeshed/meshes/abdomen.dae scale=0.06 0.06 0.06
- link neck_yaw: geometry visual mesh filename=package://rostango/models/humanMeshed/meshes/neck.dae scale=0.06 0.06 0.06
- link right_clavicle_yaw: geometry visual mesh filename=package://rostango/models/humanMeshed/meshes/rightClavicle.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 scale=0.06 0.06 0.06
- link right_elbow_yaw: geometry visual mesh filename=package://rostango/models/humanMeshed/meshes/rightForearm.d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 scale=0.062 0.06 0.06
- link right_foot_yaw: geometry visual mesh filename=package://rostango/models/humanMeshed/meshes/rightFoot.dae scale=0.06 0.06 0.06
- link right_hand_yaw: geometry visual mesh filename=package://rostango/models/humanMeshed/meshes/rightHand.dae scale=0.06 0.06 0.06
- link right_knee_yaw: geometry visual mesh filename=package://rostango/models/humanMeshed/meshes/rightShin.dae scale=0.06 0.06 0.06
- link right_shoulder_yaw: geometry visual mesh filename=package://rostango/models/humanMeshed/meshes/rightBicep.dae scale=0.07 0.06 0.06
- link right_thigh_yaw: geometry visual mesh filename=package://rostango/models/humanMeshed/meshes/rightThigh.dae scale=0.06 0.06 0.06
